Commit message: isaac version increase

File: jazzy_ws/src/grr_description/grreg.urdf (robot description, URDF)
Before this commit: robot test_robot_2026, 55 links, 54 joints
Links:
- added link usb_camera_front_link, mass 0.5; visual mesh filename=package://grr_description/meshes/camera.stl scale=0.001 0.001 0.001
- added link usb_camera_left_link, mass 0.5; visual mesh filename=package://grr_description/meshes/camera.stl scale=0.001 0.001 0.001
- added link usb_camera_right_link, mass 0.5; visual mesh filename=package://grr_description/meshes/camera.stl scale=0.001 0.001 0.001
- link chassis_link: geometry visual mesh filename=package://grr_description/meshes/drivebase.stl scale=1 1 1
- link front_left_mecanum_link: geometry visual mesh filename=package://grr_description/meshes/mecanum_wheel_1.stl scale=0.001 0.001 0.001
- link front_left_roller_0: geometry visual mesh filename=package://grr_description/meshes/mecanum_roller.stl scale=0.001 0.001 0.001
- link front_left_roller_1: geometry visual mesh filename=package://grr_description/meshes/mecanum_roller.stl scale=0.001 0.001 0.001
- link front_left_roller_2: geometry visual mesh filename=package://grr_description/meshes/mecanum_roller.stl scale=0.001 0.001 0.001
- link front_left_roller_3: geometry visual mesh filename=package://grr_description/meshes/mecanum_roller.stl scale=0.001 0.001 0.001
- link front_left_roller_4: geometry visual mesh filename=package://grr_description/meshes/mecanum_roller.stl scale=0.001 0.001 0.001
- link front_left_roller_5: geometry visual mesh filename=package://grr_description/meshes/mecanum_roller.stl scale=0.001 0.001 0.001
- link front_left_roller_6: geometry visual mesh filename=package://grr_description/meshes/mecanum_roller.stl scale=0.001 0.001 0.001
- link front_left_roller_7: geometry visual mesh filename=package://grr_description/meshes/mecanum_roller.stl scale=0.001 0.001 0.001
- link front_right_mecanum_link: geometry visual mesh filename=package://grr_description/meshes/mecanum_wheel_2.stl scale=0.001 0.001 0.001
- link front_right_roller_0: geometry visual mesh filename=package://grr_description/meshes/mecanum_roller.stl scale=0.001 0.001 0.001
- link front_right_roller_1: geometry visual mesh filename=package://grr_description/meshes/mecanum_roller.stl scale=0.001 0.001 0.001
- link front_right_roller_2: geometry visual mesh filename=package://grr_description/meshes/mecanum_roller.stl scale=0.001 0.001 0.001
- link front_right_roller_3: geometry visual mesh filename=package://grr_description/meshes/mecanum_roller.stl scale=0.001 0.001 0.001
- link front_right_roller_4: geometry visual mesh filename=package://grr_description/meshes/mecanum_roller.stl scale=0.001 0.001 0.001
- link front_right_roller_5: geometry visual mesh filename=package://grr_description/meshes/mecanum_roller.stl scale=0.001 0.001 0.001
- link front_right_roller_6: geometry visual mesh filename=package://grr_description/meshes/mecanum_roller.stl scale=0.001 0.001 0.001
- link front_right_roller_7: geometry visual mesh filename=package://grr_description/meshes/mecanum_roller.stl scale=0.001 0.001 0.001
- link intake_link: geometry visual mesh filename=package://grr_description/meshes/intake.stl scale=1 1 1
- link intake_roller_1_link: geometry visual mesh filename=package://grr_description/meshes/intake_roller.stl scale=1 1 1
- link intake_roller_2_link: geometry visual mesh filename=package://grr_description/meshes/intake_roller.stl scale=1 1 1
- link left_bin_grabber_base_link: geometry visual mesh filename=package://grr_description/meshes/bingrableft_bottom.stl scale=0.001 0.001 0.001
- link left_bin_grabber_finger_link: geometry visual mesh filename=package://grr_description/meshes/bingrableft_top.stl scale=0.001 0.001 0.001
- link left_bin_grabber_pivot_link: geometry visual mesh filename=package://grr_description/meshes/bingrableft_middle.stl scale=0.001 0.001 0.001
- link rear_left_mecanum_link: geometry visual mesh filename=package://grr_description/meshes/mecanum_wheel_2.stl scale=0.001 0.001 0.001
- link rear_left_roller_0: geometry visual mesh filename=package://grr_description/meshes/mecanum_roller.stl scale=0.001 0.001 0.001
- link rear_left_roller_1: geometry visual mesh filename=package://grr_description/meshes/mecanum_roller.stl scale=0.001 0.001 0.001
- link rear_left_roller_2: geometry visual mesh filename=package://grr_description/meshes/mecanum_roller.stl scale=0.001 0.001 0.001
- link rear_left_roller_3: geometry visual mesh filename=package://grr_description/meshes/mecanum_roller.stl scale=0.001 0.001 0.001
- link rear_left_roller_4: geometry visual mesh filename=package://grr_description/meshes/mecanum_roller.stl scale=0.001 0.001 0.001
- link rear_left_roller_5: geometry visual mesh filename=package://grr_description/meshes/mecanum_roller.stl scale=0.001 0.001 0.001
- link rear_left_roller_6: geometry visual mesh filename=package://grr_description/meshes/mecanum_roller.stl scale=0.001 0.001 0.001
- link rear_left_roller_7: geometry visual mesh filename=package://grr_description/meshes/mecanum_roller.stl scale=0.001 0.001 0.001
- link rear_right_mecanum_link: geometry visual mesh filename=package://grr_description/meshes/mecanum_wheel_1.stl scale=0.001 0.001 0.001
- link rear_right_roller_0: geometry visual mesh filename=package://grr_description/meshes/mecanum_roller.stl scale=0.001 0.001 0.001
- link rear_right_roller_1: geometry visual mesh filename=package://grr_description/meshes/mecanum_roller.stl scale=0.001 0.001 0.001
- link rear_right_roller_2: geometry visual mesh filename=package://grr_description/meshes/mecanum_roller.stl scale=0.001 0.001 0.001
- link rear_right_roller_3: geometry visual mesh filename=package://grr_description/meshes/mecanum_roller.stl scale=0.001 0.001 0.001
- link rear_right_roller_4: geometry visual mesh filename=package://grr_description/meshes/mecanum_roller.stl scale=0.001 0.001 0.001
- link rear_right_roller_5: geometry visual mesh filename=package://grr_description/meshes/mecanum_roller.stl scale=0.001 0.001 0.001
- link rear_right_roller_6: geometry visual mesh filename=package://grr_description/meshes/mecanum_roller.stl scale=0.001 0.001 0.001
- link rear_right_roller_7: geometry visual mesh filename=package://grr_description/meshes/mecanum_roller.stl scale=0.001 0.001 0.001
- link right_bin_grabber_base_link: geometry visual mesh filename=package://grr_description/meshes/bingrabright_bottom.stl scale=0.001 0.001 0.001
- link right_bin_grabber_finger_link: geometry visual mesh filename=package://grr_description/meshes/bingrabright_top.stl scale=0.001 0.001 0.001
- link right_bin_grabber_pivot_link: geometry visual mesh filename=package://grr_description/meshes/bingrabright_middle.stl scale=0.001 0.001 0.001
- link sorter_link: geometry visual mesh filename=package://grr_description/meshes/sorter_stand.stl scale=1 1 1
- link sorter_turntable_link: geometry visual mesh filename=package://grr_description/meshes/sorter.stl scale=1 1 1
Joints:
- added joint usb_camera_front_joint: type fixed, parent chassis_link, child usb_camera_front_link, origin xyz=0.10550000000000001 0.09075000000000001 0.08 rpy=0 0 1.57075
- added joint usb_camera_left_joint: type fixed, parent chassis_link, child usb_camera_left_link, origin xyz=0 -0.11075 0.06 rpy=0 0 0
- added joint usb_camera_right_joint: type fixed, parent chassis_link, child usb_camera_right_link, origin xyz=0 0.11075 0.06 rpy=0 0 3.1415
- joint front_left_mecanum_joint: origin xyz=0.09 0.10075 0 rpy=0 -1.5707963267948966 0 -> xyz=0.0855 0.10075 -0.011 rpy=0 0 0
- joint front_left_roller_0_joint: axis 0.0 0.0 1.0 -> 0.0 1.0 0.0
- joint front_left_roller_1_joint: axis 0.0 0.0 1.0 -> 0.0 1.0 0.0
- joint front_left_roller_2_joint: axis 0.0 0.0 1.0 -> 0.0 1.0 0.0
- joint front_left_roller_3_joint: axis 0.0 0.0 1.0 -> 0.0 1.0 0.0
- joint front_left_roller_4_joint: axis 0.0 0.0 1.0 -> 0.0 1.0 0.0
- joint front_left_roller_5_joint: axis 0.0 0.0 1.0 -> 0.0 1.0 0.0
- joint front_left_roller_6_joint: axis 0.0 0.0 1.0 -> 0.0 1.0 0.0
- joint front_left_roller_7_joint: axis 0.0 0.0 1.0 -> 0.0 1.0 0.0
- joint front_right_mecanum_joint: origin xyz=0.09 -0.10075 0 rpy=0 -1.5707963267948966 0 -> xyz=0.0855 -0.10075 -0.011 rpy=0 0 0
- joint front_right_roller_0_joint: axis 0.0 0.0 1.0 -> 0.0 1.0 0.0
- joint front_right_roller_1_joint: axis 0.0 0.0 1.0 -> 0.0 1.0 0.0
- joint front_right_roller_2_joint: axis 0.0 0.0 1.0 -> 0.0 1.0 0.0
- joint front_right_roller_3_joint: axis 0.0 0.0 1.0 -> 0.0 1.0 0.0
- joint front_right_roller_4_joint: axis 0.0 0.0 1.0 -> 0.0 1.0 0.0
- joint front_right_roller_5_joint: axis 0.0 0.0 1.0 -> 0.0 1.0 0.0
- joint front_right_roller_6_joint: axis 0.0 0.0 1.0 -> 0.0 1.0 0.0
- joint front_right_roller_7_joint: axis 0.0 0.0 1.0 -> 0.0 1.0 0.0
- joint left_bin_grabber_pivot_joint: axis 0 1 0 -> 0 -1 0
- joint rear_left_mecanum_joint: axis 0.0 1.0 0.0  -> 0.0 -1.0 0.0 ; origin xyz=-0.09 0.10075 0 rpy=0 -1.5707963267948966 0 -> xyz=-0.0855 0.10075 -0.011 rpy=0 0 3.141592653589793
- joint rear_left_roller_0_joint: axis 0.0 0.0 1.0 -> 0.0 1.0 0.0
- joint rear_left_roller_1_joint: axis 0.0 0.0 1.0 -> 0.0 1.0 0.0
- joint rear_left_roller_2_joint: axis 0.0 0.0 1.0 -> 0.0 1.0 0.0
- joint rear_left_roller_3_joint: axis 0.0 0.0 1.0 -> 0.0 1.0 0.0
- joint rear_left_roller_4_joint: axis 0.0 0.0 1.0 -> 0.0 1.0 0.0
- joint rear_left_roller_5_joint: axis 0.0 0.0 1.0 -> 0.0 1.0 0.0
- joint rear_left_roller_6_joint: axis 0.0 0.0 1.0 -> 0.0 1.0 0.0
- joint rear_left_roller_7_joint: axis 0.0 0.0 1.0 -> 0.0 1.0 0.0
- joint rear_right_mecanum_joint: axis 0.0 1.0 0.0  -> 0.0 -1.0 0.0 ; origin xyz=-0.09 -0.10075 0 rpy=0 -1.5707963267948966 0 -> xyz=-0.0855 -0.10075 -0.011 rpy=0 0 3.141592653589793
- joint rear_right_roller_0_joint: axis 0.0 0.0 1.0 -> 0.0 1.0 0.0
- joint rear_right_roller_1_joint: axis 0.0 0.0 1.0 -> 0.0 1.0 0.0
- joint rear_right_roller_2_joint: axis 0.0 0.0 1.0 -> 0.0 1.0 0.0
- joint rear_right_roller_3_joint: axis 0.0 0.0 1.0 -> 0.0 1.0 0.0
- joint rear_right_roller_4_joint: axis 0.0 0.0 1.0 -> 0.0 1.0 0.0
- joint rear_right_roller_5_joint: axis 0.0 0.0 1.0 -> 0.0 1.0 0.0
- joint rear_right_roller_6_joint: axis 0.0 0.0 1.0 -> 0.0 1.0 0.0
- joint rear_right_roller_7_joint: axis 0.0 0.0 1.0 -> 0.0 1.0 0.0
- joint zed21_camera_link_joint: origin xyz=0 0 0 rpy=0.2617916666666667 1.57075 0 -> xyz=0.0855 -0.09075000000000001 0.125 rpy=1.57075 0 0.2617916666666667

File: jazzy_ws/src/grr_description/urdf/parts/bin_grabber.xacro (robot description, xacro)
@@ -10,10 +10,10 @@
         <material name="yellow"/>
         </visual>
-        <collision>
+        <!-- <collision>
         <origin xyz="0 0 0" rpy="0 0 0"/>
         <geometry>
             <box size="0.1 0.1 0.1"/>
         </geometry>
-        </collision>
+        </collision> -->
     </link>
     <joint name="${prefix}_bin_grabber_base_link" type="fixed">
@@ -30,10 +30,10 @@
         <material name="red"/>
         </visual>
-        <collision>
+        <!-- <collision>
         <origin xyz="0 0 0" rpy="0 0 0"/>
         <geometry>
             <box size="0.1 0.1 0.1"/>
         </geometry>
-        </collision>
+        </collision> -->
     </link>
     <joint name="${prefix}_bin_grabber_pivot_joint" type="revolute">
@@ -41,5 +41,5 @@
         <child link="${prefix}_bin_grabber_pivot_link"/>
         <origin xyz="0.0 0.005 0" rpy="0 0 0"/>
-        <axis xyz="0 1 0"/>
+        <axis xyz="0 ${reverse} 0"/>
         <limit lower="-0.35" upper="0.044" effort="10" velocity="0.5"/>
     </joint>
@@ -52,10 +52,10 @@
         <material name="blue"/>
         </visual>
-        <collision>
+        <!-- <collision>
         <origin xyz="0 0 0" rpy="0 0 0"/>
         <geometry>
             <box size="0.1 0.1 0.1"/>
         </geometry>
-        </collision>
+        </collision> -->
     </link>
     <joint name="${prefix}_bin_grabber_finger_joint" type="revolute">

File: jazzy_ws/src/grr_description/urdf/parts/chassis.xacro (robot description, xacro)
@@ -13,10 +13,10 @@
         <!-- <material name="blue"/> -->
       </visual>
-      <collision>
+      <!-- <collision>
         <origin xyz="0 0 0" rpy="0 0 0"/>
         <geometry>
           <box size="${length} ${width} ${height/2}"/>
         </geometry>
-      </collision>
+      </collision> -->
     </link>
     <joint name="chassis_joint" type="fixed">

File: jazzy_ws/src/grr_description/urdf/parts/intake.xacro (robot description, xacro)
@@ -10,10 +10,10 @@
         <material name="yellow"/>
         </visual>
-        <collision>
+        <!-- <collision>
         <origin xyz="0 0 0" rpy="0 0 0"/>
         <geometry>
             <box size="0.1 0.1 0.1"/>
         </geometry>
-        </collision>
+        </collision> -->
     </link>
     <joint name="intake_joint" type="fixed">
@@ -30,10 +30,10 @@
         <material name="red"/>
         </visual>
-        <collision>
+        <!-- <collision>
         <origin xyz="0 0 0" rpy="0 0 0"/>
         <geometry>
             <box size="0.1 0.1 0.1"/>
         </geometry>
-        </collision>
+        </collision> -->
     </link>
     <joint name="intake_roller_1_joint" type="continuous">
@@ -51,10 +51,10 @@
         <material name="red"/>
         </visual>
-        <collision>
+        <!-- <collision>
         <origin xyz="0 0 0" rpy="0 0 0"/>
         <geometry>
             <box size="0.1 0.1 0.1"/>
         </geometry>
-        </collision>
+        </collision> -->
     </link>
     <joint name="intake_roller_2_joint" type="continuous">

File: jazzy_ws/src/grr_description/urdf/parts/mecanum_roller.xacro (robot description, xacro)
@@ -32,10 +32,10 @@
         <material name="grey"/>
       </visual>
-      <collision>
+      <!-- <collision>
         <origin xyz="0 0 0" rpy="0 0 0"/>
         <geometry>
           <mesh filename="package://grr_description/meshes/mecanum_roller.stl" scale="0.001 0.001 0.001"/>
         </geometry>
-      </collision>
+      </collision> -->
       <xacro:inertial_cylinder mass="0.07" radius="${roller_cylinder_radius}" length="${roller_length}">
         <origin xyz="0 0 0" rpy="0 0 0"/>
@@ -46,5 +46,5 @@
       <parent link="${name}_mecanum_link"/>
       <child link="${name}_roller_${number}"/>
-      <axis xyz="0.0 0.0 1.0"/>
+      <axis xyz="0.0 1.0 0.0"/>
     </joint>
   </xacro:macro>

File: jazzy_ws/src/grr_description/urdf/parts/mecanum_wheel.xacro (robot description, xacro)
@@ -4,5 +4,5 @@
     <link name="${name}_mecanum_link">
       <xacro:inertial_cylinder mass="${mass+1}" length="${width}" radius="${radius}">
-        <origin xyz="0 0 0" rpy="0 ${pi/2} 0"/>
+        <origin xyz="0 0 0" rpy="0 ${flip} 0"/>
       </xacro:inertial_cylinder>
       <visual>
@@ -13,13 +13,13 @@
         <material name="orange"/>
       </visual>
-      <collision>
+      <!-- <collision>
         <origin xyz="0 0 0" rpy="0 0 0"/>
         <geometry>
           <cylinder radius="${radius}" length="${width}"/>
         </geometry>
-      </collision>
+      </collision> -->
     </link>
     <joint name="${name}_mecanum_joint" type="continuous">
-      <origin xyz="${pos_x} ${pos_y} ${pos_z}" rpy="0 ${flip} 0"/>
+      <origin xyz="${pos_x} ${pos_y} ${pos_z}" rpy="0 0 ${flip}"/>
       <parent link="chassis_link"/>
       <child link="${name}_mecanum_link"/>

File: jazzy_ws/src/grr_description/urdf/parts/sorter.xacro (robot description, xacro)
@@ -10,10 +10,10 @@
         <material name="yellow"/>
         </visual>
-        <collision>
+        <!-- <collision>
         <origin xyz="0 0 0" rpy="0 0 0"/>
         <geometry>
             <box size="0.1 0.1 0.1"/>
         </geometry>
-        </collision>
+        </collision> -->
     </link>
     <joint name="sorter_joint" type="fixed">
@@ -30,10 +30,10 @@
         <material name="red"/>
         </visual>
-        <collision>
+        <!-- <collision>
         <origin xyz="0 0 0" rpy="0 0 0"/>
         <geometry>
             <box size="0.1 0.1 0.1"/>
         </geometry>
-        </collision>
+        </collision> -->
     </link>
     <joint name="sorter_turntable_joint" type="continuous">

File: jazzy_ws/src/grr_description/urdf/parts/usb_camera.xacro (robot description, xacro)
@@ -9,17 +9,17 @@
     <link name="usb_camera_${prefix}_link">
         <visual>
-            <origin xyz="0 0 0" rpy="0 0 -${prefix*pi/2}" />
+            <origin xyz="0 0 0" rpy="0 0 -${pi/2}" />
             <geometry>
-                <mesh filename="package://rift_description/meshes/USBCamera.stl" scale="0.001 0.001 0.001" />
+                <mesh filename="package://grr_description/meshes/camera.stl" scale="0.001 0.001 0.001" />
             </geometry>
             <material name="brown" />
         </visual>
-        <collision>
+        <!-- <collision>
             <origin xyz="0 0 0" rpy="0 0 0" />
             <geometry>
                 <box size="${camera_length} ${camera_width} ${camera_height}" />
             </geometry>
-            <!-- <material name="ghost" /> -->
-        </collision>
+            <material name="ghost" />
+        </collision> -->
         <xacro:inertial_box mass="${camera_mass}" x="${camera_length}" y="${camera_width}" z="${camera_height}">
             <origin xyz="0 0 0" rpy="0 0 0" />

File: jazzy_ws/src/grr_description/urdf/parts/zed_cam.xacro (robot description, xacro)
@@ -26,9 +26,9 @@
         <material name="zed2i_mat" />
       </visual>
-      <collision>
+      <!-- <collision>
         <geometry>
           <box size="${height} ${baseline} ${height}"/>
         </geometry>
-      </collision>
+      </collision> -->
     </link>
     <joint name="zed_camera_center_joint" type="fixed">

File: jazzy_ws/src/grr_description/urdf/robots/grreg.urdf.xacro (robot description, xacro)
@@ -13,4 +13,5 @@
   <xacro:include filename="$(find grr_description)/urdf/parts/zed_macro.xacro"/>
   <xacro:include filename="$(find grr_description)/urdf/control/drive.xacro"/>
+  <xacro:include filename="$(find grr_description)/urdf/parts/usb_camera.xacro"/>
   <!-- Properties -->
   <xacro:property name="chassis_length" value="0.18" />
@@ -22,7 +23,7 @@
   <xacro:property name="wheel_weight" value="0.136" />
   <xacro:property name="wheel_offset" value="0" />
-  <xacro:property name="wheel_joint_pos_x" value="0.09" />
+  <xacro:property name="wheel_joint_pos_x" value="0.0855" />
   <xacro:property name="wheel_joint_pos_y" value="0.10075" />
-  <xacro:property name="wheel_joint_pos_z" value="0.07793" />
+  <xacro:property name="wheel_joint_pos_z" value="0.011" />
   <xacro:property name="roller_total" value="8" />
   <xacro:property name="roller_middle_radius" value="${0.01621/2}" />
@@ -42,8 +43,8 @@
     radius="${wheel_radius}"
     width="${wheel_thickness}"
-    flip="-${pi/2}"
+    flip="${0}"
     pos_x="${wheel_joint_pos_x + wheel_offset}"
     pos_y="${wheel_joint_pos_y}"
-    pos_z="-${0}"
+    pos_z="-${wheel_joint_pos_z}"
     mass="${wheel_weight}"
   />
@@ -53,8 +54,8 @@
     radius="${wheel_radius}"
     width="${wheel_thickness}"
-    flip="-${pi/2}"
+    flip="${pi}"
     pos_x="-${wheel_joint_pos_x + wheel_offset}"
     pos_y="-${wheel_joint_pos_y}"
-    pos_z="-${0}"
+    pos_z="-${wheel_joint_pos_z}"
     mass="${wheel_weight}"
   />
@@ -64,8 +65,8 @@
     radius="${wheel_radius}"
     width="${wheel_thickness}"
-    flip="-${pi/2}"
+    flip="${pi}"
     pos_x="-${wheel_joint_pos_x + wheel_offset}"
     pos_y="${wheel_joint_pos_y}"
-    pos_z="-${0}"
+    pos_z="-${wheel_joint_pos_z}"
     mass="${wheel_weight}"
   />
@@ -75,8 +76,8 @@
     radius="${wheel_radius}"
     width="${wheel_thickness}"
-    flip="-${pi/2}"
+    flip="${0}"
     pos_x="${wheel_joint_pos_x + wheel_offset}"
     pos_y="-${wheel_joint_pos_y}"
-    pos_z="-${0}"
+    pos_z="-${wheel_joint_pos_z}"
     mass="${wheel_weight}"
   />
@@ -100,9 +101,18 @@
     parent="chassis_link">
     <origin
-        xyz="0 0 0"
-        rpy="${3.1415/12} ${3.1415/2} 0" />
+        xyz="${wheel_joint_pos_x} -${wheel_joint_pos_y-0.01} 0.125"
+        rpy="${3.1415/2} 0 ${3.1415/12}" />
     <gnss_origin
         xyz="0 0 0"
         rpy="0 0 0" />
   </xacro:zed_camera>
+  <xacro:usb_camera prefix="right" parent="chassis_link">
+    <origin xyz="0 ${wheel_joint_pos_y+0.01} 0.06" rpy="0 0 ${3.1415}"/>
+  </xacro:usb_camera>
+  <xacro:usb_camera prefix="left" parent="chassis_link">
+    <origin xyz="0 -${wheel_joint_pos_y+0.01} 0.06" rpy="0 0 0"/>
+  </xacro:usb_camera>
+  <xacro:usb_camera prefix="front" parent="chassis_link">
+    <origin xyz="${wheel_joint_pos_x+0.02} ${wheel_joint_pos_y-0.01} 0.08" rpy="0 0 ${3.1415/2}"/>
+  </xacro:usb_camera>
 </robot>
