Commit message: can tweaks

File: jazzy_ws/src/grr_description/urdf/control/drive.xacro (robot description, xacro)
@@ -3,8 +3,9 @@
   <ros2_control name="gregg" type="system">
     <hardware>
-      <plugin>grr_hardware/IsaacDriveHardware</plugin>
+      <!-- <plugin>grr_hardware/IsaacDriveHardware</plugin> -->
+      <plugin>grr_hardware/CanInterface</plugin>
       <param name="example_param_hw_start_duration_sec">3.0</param>
       <param name="example_param_hw_stop_duration_sec">3.0</param>
-      <param name="teensy1_serial_number">3030313330356332</param>
+      <!-- <param name="teensy1_serial_number">3030313330356332</param>
       <param name="teensy1_joint_names">
         <item>front_right_mecanum_joint</item>
@@ -79,5 +80,5 @@
         <item name="PWM">9</item>
       </param>
-      <param name="teensy2_serial_number">3030313330356332</param>
+      <param name="teensy2_serial_number">3030313330356332</param> -->
     </hardware>
     <joint name="front_right_mecanum_joint">
@@ -113,5 +114,5 @@
       <state_interface name="velocity"/>
     </joint>
-    <joint name="intake_roller_1_joint">
+    <!-- <joint name="intake_roller_1_joint">
       <command_interface name="effort"/>
       <state_interface name="position"/>
@@ -147,5 +148,5 @@
       <state_interface name="position"/>
       <state_interface name="velocity"/>
-    </joint>
+    </joint> -->
   </ros2_control>
 </robot>
